File: 1xRJ45/canable.sch (EAGLE design)
At the start: 24 parts, among them J2 USB-MICROB, U2 AP2202K-3.3TRG1, U3 MCP2551

Commit message: asd
Other:
- note added: "TPS73133"
Changed lines of the file:
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@@
 <text x="262.382" y="151.13" size="2.1844" layer="94" rot="R180">2-3 terminates CAN bus</text>
 <text x="261.366" y="124.968" size="2.1844" layer="94" rot="R180">1-2 enters bootloader</text>
+<text x="116.84" y="22.86" size="1.27" layer="91">TPS73133</text>
 </plain>
 <instances>
@@
 <wire x1="139.7" y1="162.56" x2="165.1" y2="162.56" width="0.1524" layer="91"/>
 <wire x1="165.1" y1="162.56" x2="165.1" y2="165.1" width="0.1524" layer="91"/>
+<label x="139.7" y="162.56" size="1.27" layer="95" rot="R180" xref="yes"/>
 </segment>
 </net>
@@
 <wire x1="139.7" y1="160.02" x2="154.94" y2="160.02" width="0.1524" layer="91"/>
 <wire x1="154.94" y1="160.02" x2="154.94" y2="165.1" width="0.1524" layer="91"/>
-</segment>
-</net>
+<label x="139.7" y="160.02" size="1.27" layer="95" rot="R180" xref="yes"/>
+</segment>
+</net>
